File: CAD/PCB/BpodDevice/r0_5_1/BpodMainBoard_r0_5_1.brd (EAGLE design)
At the start: 146.3 x 82.2 mm, 49 parts, among them Q3 2N7000, Q4 2N7000

Commit message: Corrected the printings on the PCB for BNC I/Os and Serial ports (numbers were mixed up) and added BOM
Parts:
- BNC1: value Output_Ch2 -> Output_Ch1
- BNC2: value Output_Ch1 -> Output_Ch2
- BNC3: value Input_Ch2 -> Input_Ch1
- BNC4: value Input_Ch1 -> Input_Ch2
Connections:
- net BNC1 renamed INPUT_CH_2
- net BNC2 renamed INPUT_CH_1
- net INPUT_CH1_+: now also OPTOCOUPLER.4, R3.2; no longer OPTOCOUPLER.1, R2.2
- net INPUT_CH1_GND: now also BNC3.GND, OPTOCOUPLER.3; no longer BNC4.GND, OPTOCOUPLER.2
- net INPUT_CH2_+: now also OPTOCOUPLER.1, R2.2; no longer OPTOCOUPLER.4, R3.2
- net INPUT_CH2_GND: now also BNC4.GND, OPTOCOUPLER.2; no longer BNC3.GND, OPTOCOUPLER.3
- net OUTPUT_CH1_BNC: now also BNC1.S, Q4.D, R5.1; no longer BNC2.S, Q3.D, R4.1
- net OUTPUT_CH2_BNC: now also BNC2.S, Q3.D, R4.1; no longer BNC1.S, Q4.D, R5.1
Routing:
- net INPUT_CH2_GND: track 60.7 -> 41.6 mm
- net INPUT_CH1_GND: track 41.6 -> 60.7 mm
- net INPUT_CH2_+: track 21.2 -> 7.88 mm
- net INPUT_CH1_+: track 7.88 -> 21.2 mm
- net OUTPUT_CH2_BNC: track 21.6 -> 20.0 mm
- net OUTPUT_CH1_BNC: track 20.0 -> 21.6 mm
Changed lines of the file:
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@@
 <?xml version="1.0" encoding="utf-8"?>
 <!DOCTYPE eagle SYSTEM "eagle.dtd">
-<eagle version="9.0.1">
+<eagle version="9.1.1">
 <drawing>
 <settings>
@@
 <setting verticaltext="up"/>
 </settings>
-<grid distance="0.05" unitdist="inch" unit="inch" style="lines" multiple="1" display="yes" altdistance="0.0125" altunitdist="inch" altunit="inch"/>
+<grid distance="0.05" unitdist="inch" unit="mm" style="lines" multiple="1" display="yes" altdistance="0.0125" altunitdist="inch" altunit="mm"/>
 <layers>
 <layer number="1" name="Top" color="4" fill="1" visible="yes" active="yes"/>
@@
 <text x="60.96" y="57.4675" size="1.27" layer="21" font="vector" ratio="12" align="center">Status
 LED</text>
-<text x="14.351" y="67.945" size="1.016" layer="21" font="vector" ratio="12" align="center">Input Ch1</text>
-<text x="33.4645" y="67.945" size="1.016" layer="21" font="vector" ratio="12" align="center">Input Ch2</text>
-<text x="52.578" y="67.945" size="1.016" layer="21" font="vector" ratio="12" align="center">Output Ch1</text>
-<text x="72.1995" y="67.945" size="1.016" layer="21" font="vector" ratio="12" align="center">Output Ch2</text>
+<text x="14.351" y="67.945" size="1.016" layer="21" font="vector" ratio="12" align="center">Input Ch2</text>
+<text x="33.4645" y="67.945" size="1.016" layer="21" font="vector" ratio="12" align="center">Input Ch1</text>
+<text x="52.578" y="67.945" size="1.016" layer="21" font="vector" ratio="12" align="center">Output Ch2</text>
+<text x="72.1995" y="67.945" size="1.016" layer="21" font="vector" ratio="12" align="center">Output Ch1</text>
 <text x="130.81" y="67.945" size="1.016" layer="21" font="vector" ratio="12" align="center">State SYNC</text>
-<text x="93.0275" y="67.945" size="1.016" layer="21" font="vector" ratio="12" align="center">Serial 1</text>
-<text x="112.0775" y="67.945" size="1.016" layer="21" font="vector" ratio="12" align="center">Serial 2</text>
+<text x="93.0275" y="67.945" size="1.016" layer="21" font="vector" ratio="12" align="center">Serial 2</text>
+<text x="112.0775" y="67.945" size="1.016" layer="21" font="vector" ratio="12" align="center">Serial 1</text>
 <text x="1.5875" y="20.6375" size="2.032" layer="21" font="vector" ratio="12">Open source animal behavior measurement &amp; control</text>
 <text x="131.1275" y="13.97" size="1.016" layer="21" font="vector" ratio="12" align="center">Port 8</text>
@@
 <param name="checkStop" value="0"/>
 <param name="checkValues" value="0"/>
+<param name="checkNames" value="1"/>
+<param name="checkWireStubs" value="1"/>
+<param name="checkPolygonWidth" value="0"/>
 <param name="useDiameter" value="13"/>
 <param name="maxErrors" value="50"/>
@@
 <attribute name="VALUE" x="63.5" y="28.575" size="1.27" layer="21" ratio="12" align="center"/>
 </element>
-<element name="BNC2" library="SparkFun" package="BNC" value="Output_Ch1" x="52.578" y="71.882" smashed="yes"/>
-<element name="BNC1" library="SparkFun" package="BNC" value="Output_Ch2" x="72.136" y="71.882" smashed="yes"/>
-<element name="BNC3" library="SparkFun" package="BNC" value="Input_Ch2" x="33.274" y="71.882" smashed="yes"/>
-<element name="BNC4" library="SparkFun" package="BNC" value="Input_Ch1" x="14.224" y="71.882" smashed="yes"/>
+<element name="BNC2" library="SparkFun" package="BNC" value="Output_Ch2" x="52.578" y="71.882" smashed="yes"/>
+<element name="BNC1" library="SparkFun" package="BNC" value="Output_Ch1" x="72.136" y="71.882" smashed="yes"/>
+<element name="BNC3" library="SparkFun" package="BNC" value="Input_Ch1" x="33.274" y="71.882" smashed="yes"/>
+<element name="BNC4" library="SparkFun" package="BNC" value="Input_Ch2" x="14.224" y="71.882" smashed="yes"/>
 <element name="PORT8" library="SparkFun" package="RJ45-8" value="RJ45-8PTH" x="131.064" y="3.048"/>
 <element name="PORT7" library="SparkFun" package="RJ45-8" value="RJ45-8PTH" x="114.3" y="3.048"/>
@@
 <wire x1="25.0825" y1="41.275" x2="16.8275" y2="41.275" width="0.6096" layer="16"/>
 </signal>
-<signal name="BNC1">
+<signal name="INPUT_CH_2">
 <contactref element="BNC4" pad="S"/>
 <contactref element="R2" pad="1"/>
@@
 <wire x1="12.065" y1="46.6725" x2="12.065" y2="45.72" width="0.3048" layer="16"/>
 </signal>
-<signal name="BNC2">
+<signal name="INPUT_CH_1">
 <contactref element="BNC3" pad="S"/>
 <contactref element="R3" pad="1"/>
@@
 <wire x1="8.89" y1="74.6125" x2="8.89" y2="45.72" width="0.3048" layer="16"/>
 </signal>
-<signal name="INPUT_CH2_GND">
+<signal name="INPUT_CH1_GND">
 <contactref element="BNC3" pad="GND"/>
 <contactref element="OPTOCOUPLER" pad="3"/>
@@
 <wire x1="119.38" y1="10.16" x2="119.38" y2="5.715" width="0.3048" layer="16"/>
 <wire x1="118.03261875" y1="10.7442" x2="118.29931875" y2="10.4775" width="0.3048" layer="16"/>
-<wire x1="140.335" y1="10.4775" x2="140.2207" y2="10.5918" width="0.3048" layer="16"/>
 <wire x1="99.695" y1="11.938" x2="100.838" y2="10.795" width="0.3048" layer="16"/>
 <wire x1="100.838" y1="10.795" x2="101.47418125" y2="10.795" width="0.3048" layer="16"/>
@@
 <wire x1="87.59535" y1="58.1025" x2="87.81405" y2="57.8838" width="0.3048" layer="1"/>
 <wire x1="83.82" y1="58.1025" x2="87.59535" y2="58.1025" width="0.3048" layer="1"/>
-<wire x1="87.9475" y1="57.75035" x2="87.81405" y2="57.8838" width="0.3048" layer="16"/>
 <wire x1="93.19396875" y1="54.4576" x2="89.0524" y2="54.4576" width="0.3048" layer="16"/>
 <wire x1="89.0524" y1="54.4576" x2="88.9" y2="54.61" width="0.3048" layer="16"/>
@@
 <wire x1="110.1725" y1="48.26" x2="92.964" y2="48.26" width="0.3048" layer="1"/>
 </signal>
-<signal name="OUTPUT_CH2_BNC">
+<signal name="OUTPUT_CH1_BNC">
 <contactref element="R5" pad="1"/>
 <contactref element="Q4" pad="D"/>
@@
 <wire x1="76.2" y1="71.4375" x2="75.7555" y2="71.882" width="0.3048" layer="1"/>
 </signal>
-<signal name="OUTPUT_CH1_BNC">
+<signal name="OUTPUT_CH2_BNC">
 <contactref element="BNC2" pad="S"/>
 <contactref element="R4" pad="1"/>
@@
 <wire x1="61.595" y1="67.945" x2="61.595" y2="62.865" width="0.3048" layer="16"/>
 </signal>
-<signal name="INPUT_CH1_GND">
+<signal name="INPUT_CH2_GND">
 <contactref element="OPTOCOUPLER" pad="2"/>
 <contactref element="BNC4" pad="GND"/>
@@
 <wire x1="11.684" y1="48.641" x2="12.065" y2="48.26" width="0.3048" layer="16"/>
 </signal>
-<signal name="INPUT_CH1_+">
+<signal name="INPUT_CH2_+">
 <contactref element="R2" pad="2"/>
 <contactref element="OPTOCOUPLER" pad="1"/>
@@
 <wire x1="16.51" y1="34.6075" x2="16.51" y2="36.83" width="0.3048" layer="16"/>
 </signal>
-<signal name="INPUT_CH2_+">
+<signal name="INPUT_CH1_+">
 <contactref element="OPTOCOUPLER" pad="4"/>
 <contactref element="R3" pad="2"/>
@@
 </signal>
 </signals>
+<mfgpreviewcolors>
+<mfgpreviewcolor name="soldermaskcolor" color="0xC8008000"/>
+<mfgpreviewcolor name="silkscreencolor" color="0xFFFEFEFE"/>
+<mfgpreviewcolor name="backgroundcolor" color="0xFF282828"/>
+<mfgpreviewcolor name="coppercolor" color="0xFFFFBF00"/>
+<mfgpreviewcolor name="substratecolor" color="0xFF786E46"/>
+</mfgpreviewcolors>
 </board>
 </drawing>
