File: CAD/PCB/BpodDevice/r0_5_1/BpodMainBoard_r0_5_1.sch (EAGLE design)
At the start: 48 parts, among them Q3 2N7000, Q4 2N7000

Commit message: Corrected the printings on the PCB for BNC I/Os and Serial ports (numbers were mixed up) and added BOM
Parts:
- BNC1: value Output_Ch2 -> Output_Ch1
- BNC2: value Output_Ch1 -> Output_Ch2
- BNC3: value Input_Ch2 -> Input_Ch1
- BNC4: value Input_Ch1 -> Input_Ch2
Connections:
- net BNC1 renamed INPUT_CH_2
- net BNC2 renamed INPUT_CH_1
- net INPUT_CH1_+: now also OPTOCOUPLER.4, R3.2; no longer OPTOCOUPLER.1, R2.2
- net INPUT_CH1_GND: now also BNC3.GND, OPTOCOUPLER.3; no longer BNC4.GND, OPTOCOUPLER.2
- net INPUT_CH2_+: now also OPTOCOUPLER.1, R2.2; no longer OPTOCOUPLER.4, R3.2
- net INPUT_CH2_GND: now also BNC4.GND, OPTOCOUPLER.2; no longer BNC3.GND, OPTOCOUPLER.3
- net OUTPUT_CH1_BNC: now also BNC1.OUT, Q4.D, R5.1; no longer BNC2.OUT, Q3.D, R4.1
- net OUTPUT_CH2_BNC: now also BNC2.OUT, Q3.D, R4.1; no longer BNC1.OUT, Q4.D, R5.1
Changed lines of the file:
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@@
 <?xml version="1.0" encoding="utf-8"?>
 <!DOCTYPE eagle SYSTEM "eagle.dtd">
-<eagle version="9.0.1">
+<eagle version="9.1.1">
 <drawing>
 <settings>
@@
 <parts>
 <part name="VALVE_REGISTER" library="ic-package" deviceset="DIL20" device="" value="TPIC6A595"/>
-<part name="BNC2" library="SparkFun" deviceset="BNC" device="PTH" value="Output_Ch1"/>
-<part name="BNC1" library="SparkFun" deviceset="BNC" device="PTH" value="Output_Ch2"/>
-<part name="BNC3" library="SparkFun" deviceset="BNC" device="PTH" value="Input_Ch2"/>
-<part name="BNC4" library="SparkFun" deviceset="BNC" device="PTH" value="Input_Ch1"/>
+<part name="BNC2" library="SparkFun" deviceset="BNC" device="PTH" value="Output_Ch2"/>
+<part name="BNC1" library="SparkFun" deviceset="BNC" device="PTH" value="Output_Ch1"/>
+<part name="BNC3" library="SparkFun" deviceset="BNC" device="PTH" value="Input_Ch1"/>
+<part name="BNC4" library="SparkFun" deviceset="BNC" device="PTH" value="Input_Ch2"/>
 <part name="PORT8" library="SparkFun" deviceset="RJ45-8" device="PTH"/>
 <part name="PORT7" library="SparkFun" deviceset="RJ45-8" device="PTH"/>
@@
 </busses>
 <nets>
-<net name="BNC1" class="0">
+<net name="INPUT_CH_2" class="0">
 <segment>
 <wire x1="289.56" y1="193.04" x2="287.02" y2="193.04" width="0.1524" layer="91"/>
@@
 </segment>
 </net>
-<net name="BNC2" class="0">
+<net name="INPUT_CH_1" class="0">
 <segment>
 <pinref part="BNC3" gate="G$1" pin="OUT"/>
@@
 </segment>
 </net>
-<net name="INPUT_CH2_GND" class="0">
+<net name="INPUT_CH1_GND" class="0">
 <segment>
 <wire x1="294.64" y1="165.1" x2="294.64" y2="162.56" width="0.1524" layer="91"/>
@@
 </segment>
 </net>
-<net name="OUTPUT_CH2_BNC" class="0">
+<net name="OUTPUT_CH1_BNC" class="0">
 <segment>
 <pinref part="R5" gate="G$1" pin="1"/>
@@
 </segment>
 </net>
-<net name="OUTPUT_CH1_BNC" class="0">
+<net name="OUTPUT_CH2_BNC" class="0">
 <segment>
 <pinref part="BNC2" gate="G$1" pin="OUT"/>
@@
 </segment>
 </net>
-<net name="INPUT_CH1_GND" class="0">
+<net name="INPUT_CH2_GND" class="0">
 <segment>
 <pinref part="OPTOCOUPLER" gate="G$1" pin="2"/>
@@
 </segment>
 </net>
-<net name="INPUT_CH1_+" class="0">
+<net name="INPUT_CH2_+" class="0">
 <segment>
 <pinref part="R2" gate="G$1" pin="2"/>
@@
 </segment>
 </net>
-<net name="INPUT_CH2_+" class="0">
+<net name="INPUT_CH1_+" class="0">
 <segment>
 <pinref part="OPTOCOUPLER" gate="G$1" pin="4"/>
